File: 2002-beacon.sch (KiCad schematic (older format))
At the start: 16 parts, among them J3 Barrel_Jack, Q1 2N3904, SW1 SW_SPST, U1 L7805, U2 ATtiny85-20PU

Commit message: Layout for rev2 done
Parts:
- removed C1, C2: CP1, Capacitor_THT:CP_Radial_D5.0mm_P2.00mm, symbol Device:CP1
- removed J3: Barrel_Jack, Connector_BarrelJack:BarrelJack_CUI_PJ-102AH_Horizontal, symbol Connector:Barrel_Jack
- removed U1: L7805, Package_TO_SOT_THT:TO-220-3_Horizontal_TabUp, symbol Regulator_Linear:L7805
- added C1, C3: C, Capacitor_THT:CP_Radial_D5.0mm_P2.00mm, symbol Device:C
- added D3: LED, LED_THT:LED_D3.0mm_Horizontal_O3.81mm_Z6.0mm, symbol Device:LED
- added J1: USB_B, Connector_USB:USB_Micro-B_Molex-105017-0001, symbol Connector:USB_B
- added Q2: 2N3904, Package_TO_SOT_THT:TO-92_Inline, symbol Transistor_BJT:2N3904
- added R4: 74, Resistor_THT:R_Axial_DIN0204_L3.6mm_D1.6mm_P7.62mm_Horizontal, symbol Device:R_US
- added R5: 470, Resistor_THT:R_Axial_DIN0204_L3.6mm_D1.6mm_P7.62mm_Horizontal, symbol Device:R_US
- R3: value 90 -> 74
- U2: symbol MCU_Microchip_ATtiny:ATtiny85-20PU -> 2002-beacon-rescue:ATtiny85-20PU-MCU_Microchip_ATtiny
Connections:
- wire segments 26 -> 37

Commit message: Added MFN and MPN info
Parts:
- C3: MFN (none) -> Panasonic Electronic Components; MPN (none) -> ECA-1HM100I
- D1, D3: MFN (none) -> QT Brightek; MPN (none) -> QBED8160
- D2: MFN (none) -> Cree Inc.; MPN (none) -> C503B-RAN-CZ0C0AA1
- J1: MFN (none) -> Molex; MPN (none) -> 1050170001
- Q1, Q2: MFN (none) -> ON Semiconductor; MPN (none) -> 2N3904TA
- R1, R5: MFN (none) -> Stackpole Electronics Inc; MPN (none) -> CF14JT470R
- R2: MFN (none) -> Stackpole Electronics Inc; MPN (none) -> CF14JT2K00
- R3, R4: value 74 -> 75; MFN (none) -> Vishay BC Components; MPN (none) -> SFR2500007509FR500
- SW1: MFN (none) -> TE Connectivity ALCOSWITCH Switches; MPN (none) -> 1825910-7
- U2: MFN (none) -> Atmel; MPN (none) -> ATtiny85-20PU
Changed lines of the file:
@@
 F 2 "Package_DIP:DIP-8_W7.62mm" H 4050 2950 50  0001 C CIN
 F 3 "http://ww1.microchip.com/downloads/en/DeviceDoc/atmel-2586-avr-8-bit-microcontroller-attiny25-attiny45-attiny85_datasheet.pdf" H 4050 2950 50  0001 C CNN
+F 4 "Atmel" H 4050 2950 50  0001 C CNN "MFN"
+F 5 "ATtiny85-20PU" H 4050 2950 50  0001 C CNN "MPN"
 	1    4050 2950
 	1    0    0    -1
@@
 F 2 "Button_Switch_THT:SW_PUSH_6mm" H 5350 2950 50  0001 C CNN
 F 3 "~" H 5350 2950 50  0001 C CNN
+F 4 "TE Connectivity ALCOSWITCH Switches" H 5350 2950 50  0001 C CNN "MFN"
+F 5 "1825910-7" H 5350 2950 50  0001 C CNN "MPN"
 	1    5350 2950
 	1    0    0    -1
@@
 F 2 "Resistor_THT:R_Axial_DIN0204_L3.6mm_D1.6mm_P7.62mm_Horizontal" V 5390 3290 50  0001 C CNN
 F 3 "~" H 5350 3300 50  0001 C CNN
+F 4 "Stackpole Electronics Inc" V 5350 3300 50  0001 C CNN "MFN"
+F 5 "CF14JT2K00" V 5350 3300 50  0001 C CNN "MPN"
 	1    5350 3300
 	0    1    1    0
@@
 F 2 "LED_THT:LED_D3.0mm" H 5800 3300 50  0001 C CNN
 F 3 "~" H 5800 3300 50  0001 C CNN
+F 4 "Cree Inc." H 5800 3300 50  0001 C CNN "MFN"
+F 5 "C503B-RAN-CZ0C0AA1" H 5800 3300 50  0001 C CNN "MPN"
 	1    5800 3300
 	-1   0    0    1
@@
 F 2 "Package_TO_SOT_THT:TO-92_Inline" H 5500 1775 50  0001 L CIN
 F 3 "https://www.fairchildsemi.com/datasheets/2N/2N3904.pdf" H 5300 1850 50  0001 L CNN
+F 4 "ON Semiconductor" H 5300 1850 50  0001 C CNN "MFN"
+F 5 "2N3904TA" H 5300 1850 50  0001 C CNN "MPN"
 	1    5300 1850
 	0    -1   -1   0
@@
 F 2 "LED_THT:LED_D3.0mm_Horizontal_O3.81mm_Z6.0mm" H 4350 1750 50  0001 C CNN
 F 3 "~" H 4350 1750 50  0001 C CNN
+F 4 "QT Brightek" V 4350 1750 50  0001 C CNN "MFN"
+F 5 "QBED8160" V 4350 1750 50  0001 C CNN "MPN"
 	1    4350 1750
 	-1   0    0    1
@@
 F 2 "Resistor_THT:R_Axial_DIN0204_L3.6mm_D1.6mm_P7.62mm_Horizontal" V 5340 2290 50  0001 C CNN
 F 3 "~" H 5300 2300 50  0001 C CNN
+F 4 "Stackpole Electronics Inc" H 5300 2300 50  0001 C CNN "MFN"
+F 5 "CF14JT470R" H 5300 2300 50  0001 C CNN "MPN"
 	1    5300 2300
 	1    0    0    -1
@@
 P 4800 1750
 F 0 "R3" V 4595 1750 50  0000 C CNN
-F 1 "74" V 4686 1750 50  0000 C CNN
+F 1 "75" V 4686 1750 50  0000 C CNN
 F 2 "Resistor_THT:R_Axial_DIN0204_L3.6mm_D1.6mm_P7.62mm_Horizontal" V 4840 1740 50  0001 C CNN
 F 3 "~" H 4800 1750 50  0001 C CNN
+F 4 "Vishay BC Components" V 4800 1750 50  0001 C CNN "MFN"
+F 5 "SFR2500007509FR500" V 4800 1750 50  0001 C CNN "MPN"
 	1    4800 1750
 	0    1    1    0
@@
 F 2 "Connector_USB:USB_Micro-B_Molex-105017-0001" H 2800 1600 50  0001 C CNN
 F 3 " ~" H 2800 1600 50  0001 C CNN
+F 4 "Molex" H 2650 1650 50  0001 C CNN "MFN"
+F 5 "1050170001" H 2650 1650 50  0001 C CNN "MPN"
 	1    2650 1650
 	1    0    0    -1
@@
 F 2 "Package_TO_SOT_THT:TO-92_Inline" H 7550 1775 50  0001 L CIN
 F 3 "https://www.fairchildsemi.com/datasheets/2N/2N3904.pdf" H 7350 1850 50  0001 L CNN
+F 4 "ON Semiconductor" H 7350 1850 50  0001 C CNN "MFN"
+F 5 "2N3904TA" H 7350 1850 50  0001 C CNN "MPN"
 	1    7350 1850
 	0    -1   -1   0
@@
 F 2 "LED_THT:LED_D3.0mm_Horizontal_O3.81mm_Z6.0mm" H 6400 1750 50  0001 C CNN
 F 3 "~" H 6400 1750 50  0001 C CNN
+F 4 "QT Brightek" V 6400 1750 50  0001 C CNN "MFN"
+F 5 "QBED8160" V 6400 1750 50  0001 C CNN "MPN"
 	1    6400 1750
 	-1   0    0    1
@@
 P 6850 1750
 F 0 "R4" V 6645 1750 50  0000 C CNN
-F 1 "74" V 6736 1750 50  0000 C CNN
+F 1 "75" V 6736 1750 50  0000 C CNN
 F 2 "Resistor_THT:R_Axial_DIN0204_L3.6mm_D1.6mm_P7.62mm_Horizontal" V 6890 1740 50  0001 C CNN
 F 3 "~" H 6850 1750 50  0001 C CNN
+F 4 "Vishay BC Components" V 6850 1750 50  0001 C CNN "MFN"
+F 5 "SFR2500007509FR500" V 6850 1750 50  0001 C CNN "MPN"
 	1    6850 1750
 	0    1    1    0
@@
 F 2 "Resistor_THT:R_Axial_DIN0204_L3.6mm_D1.6mm_P7.62mm_Horizontal" V 7390 2290 50  0001 C CNN
 F 3 "~" H 7350 2300 50  0001 C CNN
+F 4 "Stackpole Electronics Inc" H 7350 2300 50  0001 C CNN "MFN"
+F 5 "CF14JT470R" H 7350 2300 50  0001 C CNN "MPN"
 	1    7350 2300
 	1    0    0    -1
@@
 F 2 "Capacitor_THT:CP_Radial_D5.0mm_P2.00mm" H 6438 1200 50  0001 C CNN
 F 3 "~" H 6400 1350 50  0001 C CNN
+F 4 "Panasonic Electronic Components" V 6400 1350 50  0001 C CNN "MFN"
+F 5 "ECA-1HM100I" V 6400 1350 50  0001 C CNN "MPN"
 	1    6400 1350
 	0    1    1    0
